File: PCB Design/VoltageRegulator/VoltageRegulator.kicad_pcb (KiCad board)
At the start: 2 copper layers, 55.9 x 55.9 mm, 12 parts, among them J1 Screw_Terminal_01x08, U1 LM7815_TO220, U2 LM7806_TO220

Commit message: Continued drafting report
Parts:
- removed the G*** at (127.0, 113.0)
