File: PCB Design/S_Tele/S_Tele.kicad_sch (KiCad schematic)
At the start: 33 parts, among them J1 Screw_Terminal_01x08, J2 SMA, J3 SMA, J4 SMA, J5 SMA, J6 SMA, J7 SMA, J8 Conn_01x01, U1 L7815, U2 L7805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

Commit message: PCB Rev D drafted, DRC pass
Parts:
- renumbered J8 to J2, J2 to J5, J5 to J7, J7 to J8
Connections:
- net +15VDC: now also J1.6 (Pin_6), J1.7 (Pin_7); no longer J1.2 (Pin_2), J1.3 (Pin_3)
- net GND: now also J1.1 (Pin_1), J1.2 (Pin_2), J1.3 (Pin_3); no longer J1.6 (Pin_6), J1.7 (Pin_7), J1.8 (Pin_8)
- net Vin: now also J1.8 (Pin_8); no longer J1.1 (Pin_1)
- net RFIN: now reaches C10.1, J3.1 (In), R3.1
Other:
- note added: "6/28/2023"
- note removed: "6/26/2023"
- moved on the sheet: J1

Commit message: Bill of materials added
Parts:
- C1, C2, C3, C4: footprint Capacitor_Tantalum_SMD:CP_EIA-1608-08_AVX-J -> Capacitor_Tantalum_SMD:CP_EIA-2012-12_Kemet-R
Changed lines of the file:
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@@
       (effects (font (size 1.27 1.27)) (justify left))
     )
-    (property "Footprint" "Capacitor_Tantalum_SMD:CP_EIA-1608-08_AVX-J" (at 119.38 54.61 0)
+    (property "Footprint" "Capacitor_Tantalum_SMD:CP_EIA-2012-12_Kemet-R" (at 119.38 54.61 0)
       (effects (font (size 1.27 1.27)) hide)
     )
@@
       (effects (font (size 1.27 1.27)) (justify left))
     )
-    (property "Footprint" "Capacitor_Tantalum_SMD:CP_EIA-1608-08_AVX-J" (at 50.8 54.61 0)
+    (property "Footprint" "Capacitor_Tantalum_SMD:CP_EIA-2012-12_Kemet-R" (at 50.8 54.61 0)
       (effects (font (size 1.27 1.27)) hide)
     )
@@
       (effects (font (size 1.27 1.27)) (justify left))
     )
-    (property "Footprint" "Capacitor_Tantalum_SMD:CP_EIA-1608-08_AVX-J" (at 77.47 54.61 0)
+    (property "Footprint" "Capacitor_Tantalum_SMD:CP_EIA-2012-12_Kemet-R" (at 77.47 54.61 0)
       (effects (font (size 1.27 1.27)) hide)
     )
@@
       (effects (font (size 1.27 1.27)) (justify left))
     )
-    (property "Footprint" "Capacitor_Tantalum_SMD:CP_EIA-1608-08_AVX-J" (at 92.71 54.61 0)
-      (effects (font (size 1.27 1.27)) hide)
-    )
+    (property "Footprint" "Capacitor_Tantalum_SMD:CP_EIA-2012-12_Kemet-R" (at 92.71 54.61 0)
+      (effects (font (size 1.27 1.27)) hide)
+    )
